File: electronics/driver_board/driver.brd (EAGLE design)
At the start: 160 x 100 mm, 40 parts, among them IC1 ACS711KEXLT-31AB-T, IC2 ATTINY44A-SSU, IC3 ACS711KEXLT-31AB-T, IC4 DGD0506AM10-13, IC5 DGD0506AM10-13, IC6 LMZ14201HTZ, IC7 ISO1541D, Q1 TPN3R704PL,L1Q, Q2 TPN3R704PL,L1Q, Q3 TPN3R704PL,L1Q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

Commit message: For review 2
Parts:
- added ISOLATE: (no value), rcl:R0805
- added JP1: (no value), pinhead:2X03
- added JP2: (no value), pinhead:1X06
- added U$1, U$2: XT30, parts:XT30
- moved IC7 233.5 mm to (39.4, 17.8), turned to 270 degrees
- moved C1 39.6 mm to (101.6, 14.0)
- moved C9 39.6 mm to (91.4, 12.7)
- moved IC1 39.6 mm to (127.0, 10.2)
- moved IC2 39.6 mm to (94.0, 19.1)
- moved IC3 39.6 mm to (127.0, 21.6)
- moved Q1 39.6 mm to (121.9, 16.5)
- moved Q2 39.6 mm to (121.9, 10.2)
- moved Q3 39.6 mm to (121.9, 27.9)
- moved Q4 39.6 mm to (121.9, 21.6)
- moved R10 39.6 mm to (95.2, 27.9)
- moved R12 39.6 mm to (100.3, 21.0)
- moved R13 39.6 mm to (100.3, 16.9)
- moved R17 39.6 mm to (110.5, 7.62)
- moved R18 39.6 mm to (91.4, 24.1)
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Connections:
- removed net VCC1: IC7.1
- new net N$19: IC7.2, U1.17
- new net N$23: IC7.3, U1.18
- new net N$24: IC7.1, ISOLATE.1, U1.2
- net +3V3: now also IC7.8, ISOLATE.2, JP1.2, JP2.4; no longer U1.2
- net +V_GATE: now also JP2.3
- net +V_MONITOR: now also IC2.8, JP1.1; no longer IC2.13
- net GND: now also IC7.4, IC7.5, JP1.6, JP2.5, U$2.P$1
- net I_B: now also IC2.13; no longer IC2.8
- net OUT_A: now also U$1.P$1
- net OUT_B: now also U$1.P$2
- net RESET: now also JP1.5
- net SCL: now also IC7.6, JP1.3, JP2.1; no longer U1.18
- net SDA: now also IC7.7, JP1.4, JP2.2; no longer U1.17
- net V+: now also JP2.6, U$2.P$2
Routing:
- net GND: track 44.6 -> 136.9 mm, vias 48 -> 54
- net SDA: track 32.4 -> 122.3 mm, vias 2 -> 5
- net SCL: track 34.7 -> 117.7 mm, vias 2 -> 4
- net +3V3: track 144.2 -> 221.8 mm, vias 12 -> 13
- net V+: track 23.3 -> 86.6 mm, vias 18 -> 19
- net +V_GATE: track 81.8 -> 134.8 mm
- net N$24: track 0.00 -> 45.4 mm
- net RESET: track 8.95 -> 20.5 mm, vias 2 -> 3
- net +V_MONITOR: track 35.6 -> 46.9 mm, vias 0 -> 4
- net N$19: track 0.00 -> 10.4 mm
- net N$23: track 0.00 -> 9.90 mm
- net I_B: track 44.2 -> 50.8 mm
- added copper zone on layer 1, net OUT_A
- added copper zone on layer 1, net OUT_B
Other:
- board size 160 x 100 mm -> 135.9 x 36.5 mm
