File: electronics/driver_board/driver.sch (EAGLE design)
At the start: 40 parts, among them IC1 ACS711KEXLT-31AB-T, IC2 ATTINY44A-SSU, IC3 ACS711KEXLT-31AB-T, IC4 DGD0506AM10-13, IC5 DGD0506AM10-13, IC6 LMZ14201HTZ, IC7 ISO1541D, Q1 TPN3R704PL,L1Q, Q2 TPN3R704PL,L1Q, Q3 TPN3R704PL,L1Q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

Commit message: For review 2
Parts:
- added ISOLATE: (no value), rcl:R-EU_R0805
- added JP1: (no value), pinhead:PINHD-2X3
- added JP2: (no value), pinhead:PINHD-1X6
- added U$1, U$2: XT30, parts:XT30
Connections:
- new net N$19: IC7.SDA1, U1.SDA
- new net N$23: IC7.SCL1, U1.SCL
- new net N$24: IC7.VCC1, ISOLATE.1, U1.3V
- net +3V3: now also IC7.VCC2, ISOLATE.2, JP1.2, JP2.4; no longer U1.3V
- net +V_GATE: now also JP2.3
- net +V_MONITOR: now also IC2.PA5[ADC5/DO/MISO/OC1B/PCINT5], JP1.1; no longer IC2.PA0[ADC0/AREF/PCINT0]
- net GND: now also IC7.GND1, IC7.GND2, JP1.6, JP2.5, U$2.1
- net I_B: now also IC2.PA0[ADC0/AREF/PCINT0]; no longer IC2.PA5[ADC5/DO/MISO/OC1B/PCINT5]
- net OUT_A: now also U$1.1
- net OUT_B: now also U$1.2
- net RESET: now also JP1.5
- net SCL: now also IC7.SCL2, JP1.3, JP2.1; no longer U1.SCL
- net SDA: now also IC7.SDA2, JP1.4, JP2.2; no longer U1.SDA
- net V+: now also JP2.6, U$2.2
Other:
- moved on the sheet: C9, IC2, IC7, R12, R13, R18, U1
